File: hardware/testHW/mpp_bldc_GAN.sch (EAGLE design)
At the start: 67 parts, among them IC1 ATXMEGA16A4U-MH, U1 LM3480IM3-5, U3 MIC5504-2.8YM5-TR, X1 PASSER-07, X2 PASSER-07, X3 PASSER-07, X4 PASSER-07

Commit message: testing
Parts:
- removed C16, C17: CAP TANT 22UF 25V 10% 2312, rcl:CPOL-EUC/6032-28R
- removed X1, X2, X3, X4: PASSER-07, we-symbol:PASSER-07
- added C1, C28, C29, C30, C31, C32: 10uF/25V/CC, rcl:C-EUC1206
- C5, C6, C7: device rcl:C-EUC0603 -> rcl:C-EUC0402
- R12, R13, R14, R15, R16, R17, R18, R19, R20, R21, R22: device rcl:R-EU_R0603 -> rcl:R-EU_R0402
- R2: device resistor:R-EU_R0603 -> resistor:R-EU_R0402
- RX_DIRECT: value TPSQTP19SQ -> TPSQTP11SQ; device testpad:TPSQTP19SQ -> testpad:TPSQTP11SQ
- TP7: value TPSQTP19SQ -> TPSQTP10R; device testpad:TPSQTP19SQ -> testpad:TPSQTP10R
Connections:
- net N$1 renamed PROG_JMP
- removed net RC_SIG_IC: IC1.PB0, R1.2
- new net N$4: IC1.PE2, R1.2
- net GND: now also C1.1, C28.1, C29.1, C30.1, C31.1, C32.1; no longer C16.-, C17.-
- net VCC: now also C1.2, C28.2, C29.2, C30.2, C31.2, C32.2; no longer C16.+, C17.+
Other:
- moved on the sheet: D4, R1, RX_IN_PIN
